Commit message: Added base_footprint link

File: description/robot_core.xacro (robot description, xacro)
@@ -19,4 +19,12 @@
     <!-- BASE LINK-->
     <link name = "base_link">
+    </link>
+    <!-- BASE_FOOTPRINT LINK -->
+    <joint name="base_footprint_joint" type="fixed">
+        <parent link="base_link"/>
+        <child link="base_footprint"/>
+        <origin xyz="0 0 0" rpy="0 0 0"/>
+    </joint>
+    <link name="base_footprint">
     </link>
     <!-- CHASSIS LINK-->
@@ -124,6 +132,6 @@
     <gazebo reference="caster_wheel">
         <material>Gazebo/White</material>
-        <mu1 value="0.001"/>
-        <mu2 value="0.001"/>
+        <mu1 value="0.000001"/>
+        <mu2 value="0.000001"/>
     </gazebo>
 </robot>
